File: PowerMgmt.sch (KiCad schematic (older format))
At the start: 14 parts

Commit message: fix missing regulator, add power mgmt lib
Parts:
- removed U?: MCP1700T-3002E/TT, symbol MCP1700T-3002E/TT
- added U?: MCP1700-3002E_SOT23, TO_SOT_Packages_SMD:SOT-23, symbol MCP1700-3002E_SOT23
Changed lines of the file:
@@
 LIBS:rfcom
 LIBS:maxim
-LIBS:soilsensor-cache
+LIBS:battery_management
 EELAYER 25 0
 EELAYER END
@@
 $EndComp
 $Comp
-L MCP1700T-3002E/TT U?
-U 1 1 59568C29
-P 6100 3050
-F 0 "U?" H 6200 2900 50  0000 C CNN
-F 1 "MCP1700T-3002E/TT" H 6100 3300 50  0000 C CNN
-F 2 "" H 6100 3050 50  0001 C CNN
-F 3 "" H 6100 3050 50  0000 C CNN
-	1    6100 3050
-	1    0    0    -1
-$EndComp
-$Comp
 L C C?
 U 1 1 59568C2A
@@
 NoConn ~ 3800 3750
 Connection ~ 3650 3650
+$Comp
+L MCP1700-3002E_SOT23 U?
+U 1 1 59568268
+P 6100 2950
+F 0 "U?" H 5950 3200 50  0000 C CNN
+F 1 "MCP1700-3002E_SOT23" H 5500 3100 50  0000 L CNN
+F 2 "TO_SOT_Packages_SMD:SOT-23" H 6100 3175 50  0001 C CNN
+F 3 "" H 6100 2950 50  0001 C CNN
+	1    6100 2950
+	1    0    0    -1
+$EndComp
 $EndSCHEMATC

Commit message: update power management
- add battery connector
- remove unnecessary filter
Parts:
- removed C?: 47u, symbol C
- removed L?: 6.8uH, symbol L_Small
- added J?: BATT_CONN, symbol CONN_01X02
Connections:
- net labels removed: VDDA
- wire segments 46 -> 47
Other:
- moved on the sheet: C?
Changed lines of the file:
@@
 L C C?
 U 1 1 59568C2A
-P 5700 3750
-F 0 "C?" H 5725 3850 50  0000 L CNN
-F 1 "1u" H 5725 3650 50  0000 L CNN
-F 2 "" H 5738 3600 50  0001 C CNN
-F 3 "" H 5700 3750 50  0000 C CNN
-	1    5700 3750
+P 5700 3200
+F 0 "C?" H 5725 3300 50  0000 L CNN
+F 1 "1u" H 5725 3100 50  0000 L CNN
+F 2 "" H 5738 3050 50  0001 C CNN
+F 3 "" H 5700 3200 50  0000 C CNN
+	1    5700 3200
 	1    0    0    -1
 $EndComp
@@
 L C C?
 U 1 1 59568C2B
-P 6500 3500
-F 0 "C?" H 6525 3600 50  0000 L CNN
-F 1 "1u" H 6525 3400 50  0000 L CNN
-F 2 "" H 6538 3350 50  0001 C CNN
-F 3 "" H 6500 3500 50  0000 C CNN
-	1    6500 3500
+P 6500 3200
+F 0 "C?" H 6525 3300 50  0000 L CNN
+F 1 "1u" H 6525 3100 50  0000 L CNN
+F 2 "" H 6538 3050 50  0001 C CNN
+F 3 "" H 6500 3200 50  0000 C CNN
+	1    6500 3200
 	1    0    0    -1
 $EndComp
@@
 L GND #PWR?
 U 1 1 59568C2C
-P 6100 4000
-F 0 "#PWR?" H 6100 3750 50  0001 C CNN
-F 1 "GND" H 6100 3850 50  0000 C CNN
-F 2 "" H 6100 4000 50  0000 C CNN
-F 3 "" H 6100 4000 50  0000 C CNN
-	1    6100 4000
-	1    0    0    -1
-$EndComp
-$Comp
-L L_Small L?
-U 1 1 59568C2D
-P 6750 2950
-F 0 "L?" V 6850 2950 50  0000 L CNN
-F 1 "6.8uH" V 6700 2850 50  0000 L CNN
-F 2 "" H 6750 2950 50  0001 C CNN
-F 3 "" H 6750 2950 50  0000 C CNN
-	1    6750 2950
-	0    -1   -1   0
-$EndComp
-$Comp
-L C C?
-U 1 1 59568C2E
-P 7000 3500
-F 0 "C?" H 7025 3600 50  0000 L CNN
-F 1 "47u" H 7025 3400 50  0000 L CNN
-F 2 "" H 7038 3350 50  0001 C CNN
-F 3 "" H 7000 3500 50  0000 C CNN
-	1    7000 3500
+P 6100 3600
+F 0 "#PWR?" H 6100 3350 50  0001 C CNN
+F 1 "GND" H 6100 3450 50  0000 C CNN
+F 2 "" H 6100 3600 50  0000 C CNN
+F 3 "" H 6100 3600 50  0000 C CNN
+	1    6100 3600
 	1    0    0    -1
 $EndComp
@@
 $EndComp
 $Comp
-L VDDA #PWR?
-U 1 1 59568C30
-P 7000 2750
-F 0 "#PWR?" H 7000 2600 50  0001 C CNN
-F 1 "VDDA" H 7000 2900 50  0000 C CNN
-F 2 "" H 7000 2750 50  0000 C CNN
-F 3 "" H 7000 2750 50  0000 C CNN
-	1    7000 2750
-	1    0    0    -1
-$EndComp
-$Comp
 L GND #PWR?
 U 1 1 59568C34
@@
 	5000 3050 5150 3050
 Wire Wire Line
-	5700 2950 5700 3600
+	5700 2950 5700 3050
 Wire Wire Line
 	5000 2950 5800 2950
@@
 Wire Wire Line
 	3400 3500 3400 3850
-Connection ~ 7000 2950
-Wire Wire Line
-	7000 2750 7000 3350
-Connection ~ 6500 3950
-Wire Wire Line
-	7000 3950 7000 3650
-Wire Wire Line
-	6850 2950 7000 2950
 Connection ~ 6500 2950
 Wire Wire Line
-	6500 2750 6500 3350
-Wire Wire Line
-	6400 2950 6650 2950
-Wire Wire Line
-	5700 3900 5700 3950
-Connection ~ 6100 3950
-Wire Wire Line
-	5700 3950 7000 3950
-Wire Wire Line
-	6500 3950 6500 3650
-Wire Wire Line
-	6100 3250 6100 4000
+	6500 2750 6500 3050
+Wire Wire Line
+	5700 3350 5700 3500
+Wire Wire Line
+	6500 3500 6500 3350
+Wire Wire Line
+	6100 3250 6100 3600
 Connection ~ 5400 3450
 Wire Wire Line
@@
 	1    0    0    -1
 $EndComp
+$Comp
+L CONN_01X02 J?
+U 1 1 59568744
+P 2750 4350
+F 0 "J?" H 2750 4500 50  0000 C CNN
+F 1 "BATT_CONN" V 2850 4350 50  0000 C CNN
+F 2 "" H 2750 4350 50  0001 C CNN
+F 3 "" H 2750 4350 50  0001 C CNN
+	1    2750 4350
+	-1   0    0    -1
+$EndComp
+$Comp
+L +BATT #PWR?
+U 1 1 59568804
+P 3050 4200
+F 0 "#PWR?" H 3050 4050 50  0001 C CNN
+F 1 "+BATT" H 3050 4340 50  0000 C CNN
+F 2 "" H 3050 4200 50  0000 C CNN
+F 3 "" H 3050 4200 50  0000 C CNN
+	1    3050 4200
+	1    0    0    -1
+$EndComp
+$Comp
+L GND #PWR?
+U 1 1 5956883C
+P 3050 4500
+F 0 "#PWR?" H 3050 4250 50  0001 C CNN
+F 1 "GND" H 3050 4350 50  0000 C CNN
+F 2 "" H 3050 4500 50  0000 C CNN
+F 3 "" H 3050 4500 50  0000 C CNN
+	1    3050 4500
+	1    0    0    -1
+$EndComp
+Wire Wire Line
+	2950 4300 3050 4300
+Wire Wire Line
+	3050 4300 3050 4200
+Wire Wire Line
+	2950 4400 3050 4400
+Wire Wire Line
+	3050 4400 3050 4500
+Wire Wire Line
+	6400 2950 6500 2950
+Wire Wire Line
+	5700 3500 6500 3500
+Connection ~ 6100 3500
 $EndSCHEMATC

Commit message: fix minors, make annotations
Parts:
- P1: renamed from P?; footprint (none) -> Connect:USB_Micro-B
- U3: renamed from U?; footprint (none) -> Housings_DFN_QFN:QFN-16-1EP_3x3mm_Pitch0.5mm
- gave numbers to parts that had none: 11
Changed lines of the file:
@@
 $EndDescr
 $Comp
-L USB_OTG P?
+L USB_OTG P1
 U 1 1 59568C23
 P 2900 3250
-F 0 "P?" H 3000 2900 50  0000 C CNN
+F 0 "P1" H 3000 2900 50  0000 C CNN
 F 1 "USB_OTG" H 2900 3600 50  0000 C CNN
-F 2 "" V 2850 3150 50  0001 C CNN
+F 2 "Connect:USB_Micro-B" V 2850 3150 50  0001 C CNN
 F 3 "" V 2850 3150 50  0000 C CNN
 	1    2900 3250
@@
 $EndComp
 $Comp
-L C C?
+L C C4
 U 1 1 59568C2A
 P 5700 3200
-F 0 "C?" H 5725 3300 50  0000 L CNN
+F 0 "C4" H 5725 3300 50  0000 L CNN
 F 1 "1u" H 5725 3100 50  0000 L CNN
 F 2 "" H 5738 3050 50  0001 C CNN
@@
 $EndComp
 $Comp
-L C C?
+L C C5
 U 1 1 59568C2B
 P 6500 3200
-F 0 "C?" H 6525 3300 50  0000 L CNN
+F 0 "C5" H 6525 3300 50  0000 L CNN
 F 1 "1u" H 6525 3100 50  0000 L CNN
 F 2 "" H 6538 3050 50  0001 C CNN
@@
 $EndComp
 $Comp
-L GND #PWR?
+L GND #PWR08
 U 1 1 59568C2C
 P 6100 3600
-F 0 "#PWR?" H 6100 3350 50  0001 C CNN
+F 0 "#PWR08" H 6100 3350 50  0001 C CNN
 F 1 "GND" H 6100 3450 50  0000 C CNN
 F 2 "" H 6100 3600 50  0000 C CNN
@@
 $EndComp
 $Comp
-L VDD #PWR?
+L VDD #PWR09
 U 1 1 59568C2F
 P 6500 2750
-F 0 "#PWR?" H 6500 2600 50  0001 C CNN
+F 0 "#PWR09" H 6500 2600 50  0001 C CNN
 F 1 "VDD" H 6500 2900 50  0000 C CNN
 F 2 "" H 6500 2750 50  0000 C CNN
@@
 $EndComp
 $Comp
-L GND #PWR?
+L GND #PWR010
 U 1 1 59568C34
 P 3400 3850
-F 0 "#PWR?" H 3400 3600 50  0001 C CNN
+F 0 "#PWR010" H 3400 3600 50  0001 C CNN
 F 1 "GND" H 3400 3700 50  0000 C CNN
 F 2 "" H 3400 3850 50  0000 C CNN
@@
 $EndComp
 $Comp
-L R R?
+L R R4
 U 1 1 59568C35
 P 4500 4200
-F 0 "R?" V 4580 4200 50  0000 C CNN
+F 0 "R4" V 4580 4200 50  0000 C CNN
 F 1 "1k" V 4500 4200 50  0000 C CNN
 F 2 "" V 4430 4200 50  0001 C CNN
@@
 $EndComp
 $Comp
-L R R?
+L R R5
 U 1 1 59568C36
 P 4650 4200
-F 0 "R?" V 4730 4200 50  0000 C CNN
+F 0 "R5" V 4730 4200 50  0000 C CNN
 F 1 "1k" V 4650 4200 50  0000 C CNN
 F 2 "" V 4580 4200 50  0001 C CNN
@@
 $EndComp
 $Comp
-L GND #PWR?
+L GND #PWR011
 U 1 1 59568C37
 P 4400 4550
-F 0 "#PWR?" H 4400 4300 50  0001 C CNN
+F 0 "#PWR011" H 4400 4300 50  0001 C CNN
 F 1 "GND" H 4400 4400 50  0000 C CNN
 F 2 "" H 4400 4550 50  0000 C CNN
@@
 $EndComp
 $Comp
-L R R?
+L R R6
 U 1 1 59568C38
 P 5050 4200
-F 0 "R?" V 5130 4200 50  0000 C CNN
+F 0 "R6" V 5130 4200 50  0000 C CNN
 F 1 "10k" V 5050 4200 50  0000 C CNN
 F 2 "" V 4980 4200 50  0001 C CNN
@@
 $EndComp
 $Comp
-L C C?
+L C C3
 U 1 1 59568C39
 P 5400 3750
-F 0 "C?" H 5425 3850 50  0000 L CNN
+F 0 "C3" H 5425 3850 50  0000 L CNN
 F 1 "22u" H 5425 3650 50  0000 L CNN
 F 2 "" H 5438 3600 50  0001 C CNN
@@
 $EndComp
 $Comp
-L GND #PWR?
+L GND #PWR012
 U 1 1 59568C3A
 P 5400 4000
-F 0 "#PWR?" H 5400 3750 50  0001 C CNN
+F 0 "#PWR012" H 5400 3750 50  0001 C CNN
 F 1 "GND" H 5400 3850 50  0000 C CNN
 F 2 "" H 5400 4000 50  0000 C CNN
@@
 $EndComp
 $Comp
-L BQ24075 U?
+L BQ24075 U3
 U 1 1 59568C59
 P 4400 3350
-F 0 "U?" H 4000 3950 50  0000 C CNN
+F 0 "U3" H 4000 3950 50  0000 C CNN
 F 1 "BQ24075" H 4800 2750 50  0000 C CNN
-F 2 "" H 4600 3100 50  0001 C CNN
+F 2 "Housings_DFN_QFN:QFN-16-1EP_3x3mm_Pitch0.5mm" H 4600 3100 50  0001 C CNN
 F 3 "" H 4600 3550 50  0000 C CNN
 	1    4400 3350
@@
 $EndComp
 $Comp
-L C C?
+L C C2
 U 1 1 59568C5A
 P 3400 3350
-F 0 "C?" H 3425 3450 50  0000 L CNN
+F 0 "C2" H 3425 3450 50  0000 L CNN
 F 1 "4.7u" H 3425 3250 50  0000 L CNN
 F 2 "" H 3438 3200 50  0001 C CNN
@@
 $EndComp
 $Comp
-L +BATT #PWR?
+L +BATT #PWR013
 U 1 1 59568C5B
 P 5400 3350
-F 0 "#PWR?" H 5400 3200 50  0001 C CNN
+F 0 "#PWR013" H 5400 3200 50  0001 C CNN
 F 1 "+BATT" H 5400 3490 50  0000 C CNN
 F 2 "" H 5400 3350 50  0000 C CNN
@@
 	5050 3750 5000 3750
 $Comp
-L VDD #PWR?
+L VDD #PWR014
 U 1 1 59568C69
 P 4400 2200
-F 0 "#PWR?" H 4400 2050 50  0001 C CNN
+F 0 "#PWR014" H 4400 2050 50  0001 C CNN
 F 1 "VDD" H 4400 2350 50  0000 C CNN
 F 2 "" H 4400 2200 50  0000 C CNN
@@
 $EndComp
 $Comp
-L R R?
+L R R2
 U 1 1 59568C6A
 P 4300 2400
-F 0 "R?" V 4380 2400 50  0000 C CNN
+F 0 "R2" V 4380 2400 50  0000 C CNN
 F 1 "100k" V 4300 2400 50  0000 C CNN
 F 2 "" V 4230 2400 50  0001 C CNN
@@
 $EndComp
 $Comp
-L R R?
+L R R3
 U 1 1 59568C6B
 P 4500 2400
-F 0 "R?" V 4580 2400 50  0000 C CNN
+F 0 "R3" V 4580 2400 50  0000 C CNN
 F 1 "100k" V 4500 2400 50  0000 C CNN
 F 2 "" V 4430 2400 50  0001 C CNN
@@
 Connection ~ 3650 3650
 $Comp
-L MCP1700-3002E_SOT23 U?
+L MCP1700-3002E_SOT23 U4
 U 1 1 59568268
 P 6100 2950
-F 0 "U?" H 5950 3200 50  0000 C CNN
+F 0 "U4" H 5950 3200 50  0000 C CNN
 F 1 "MCP1700-3002E_SOT23" H 5500 3100 50  0000 L CNN
 F 2 "TO_SOT_Packages_SMD:SOT-23" H 6100 3175 50  0001 C CNN
@@
 $EndComp
 $Comp
-L CONN_01X02 J?
+L CONN_01X02 J2
 U 1 1 59568744
 P 2750 4350
-F 0 "J?" H 2750 4500 50  0000 C CNN
+F 0 "J2" H 2750 4500 50  0000 C CNN
 F 1 "BATT_CONN" V 2850 4350 50  0000 C CNN
 F 2 "" H 2750 4350 50  0001 C CNN
@@
 $EndComp
 $Comp
-L +BATT #PWR?
+L +BATT #PWR015
 U 1 1 59568804
 P 3050 4200
-F 0 "#PWR?" H 3050 4050 50  0001 C CNN
+F 0 "#PWR015" H 3050 4050 50  0001 C CNN
 F 1 "+BATT" H 3050 4340 50  0000 C CNN
 F 2 "" H 3050 4200 50  0000 C CNN
@@
 $EndComp
 $Comp
-L GND #PWR?
+L GND #PWR016
 U 1 1 5956883C
 P 3050 4500
-F 0 "#PWR?" H 3050 4250 50  0001 C CNN
+F 0 "#PWR016" H 3050 4250 50  0001 C CNN
 F 1 "GND" H 3050 4350 50  0000 C CNN
 F 2 "" H 3050 4500 50  0000 C CNN
