File: PowerMgmt.sch (KiCad schematic (older format))
At the start: 13 parts, among them J2 BATT_CONN, P1 USB_OTG, U3 BQ24075, U4 MCP1700-3002E_SOT23

Commit message: update footprints
Parts:
- C2, C3, C4, C5: footprint (none) -> Capacitors_SMD:C_0805_HandSoldering
- J2: footprint (none) -> Connectors_JST:JST_PH_S2B-PH-K_02x2.00mm_Angled
- R2, R3, R4, R5, R6: footprint (none) -> Resistors_SMD:R_0805_HandSoldering
Changed lines of the file:
@@
 F 0 "C4" H 5725 3300 50  0000 L CNN
 F 1 "1u" H 5725 3100 50  0000 L CNN
-F 2 "" H 5738 3050 50  0001 C CNN
+F 2 "Capacitors_SMD:C_0805_HandSoldering" H 5738 3050 50  0001 C CNN
 F 3 "" H 5700 3200 50  0000 C CNN
 	1    5700 3200
@@
 F 0 "C5" H 6525 3300 50  0000 L CNN
 F 1 "1u" H 6525 3100 50  0000 L CNN
-F 2 "" H 6538 3050 50  0001 C CNN
+F 2 "Capacitors_SMD:C_0805_HandSoldering" H 6538 3050 50  0001 C CNN
 F 3 "" H 6500 3200 50  0000 C CNN
 	1    6500 3200
@@
 F 0 "R4" V 4580 4200 50  0000 C CNN
 F 1 "1k" V 4500 4200 50  0000 C CNN
-F 2 "" V 4430 4200 50  0001 C CNN
+F 2 "Resistors_SMD:R_0805_HandSoldering" V 4430 4200 50  0001 C CNN
 F 3 "" H 4500 4200 50  0000 C CNN
 	1    4500 4200
@@
 F 0 "R5" V 4730 4200 50  0000 C CNN
 F 1 "1k" V 4650 4200 50  0000 C CNN
-F 2 "" V 4580 4200 50  0001 C CNN
+F 2 "Resistors_SMD:R_0805_HandSoldering" V 4580 4200 50  0001 C CNN
 F 3 "" H 4650 4200 50  0000 C CNN
 	1    4650 4200
@@
 F 0 "R6" V 5130 4200 50  0000 C CNN
 F 1 "10k" V 5050 4200 50  0000 C CNN
-F 2 "" V 4980 4200 50  0001 C CNN
+F 2 "Resistors_SMD:R_0805_HandSoldering" V 4980 4200 50  0001 C CNN
 F 3 "" H 5050 4200 50  0000 C CNN
 	1    5050 4200
@@
 F 0 "C3" H 5425 3850 50  0000 L CNN
 F 1 "22u" H 5425 3650 50  0000 L CNN
-F 2 "" H 5438 3600 50  0001 C CNN
+F 2 "Capacitors_SMD:C_0805_HandSoldering" H 5438 3600 50  0001 C CNN
 F 3 "" H 5400 3750 50  0000 C CNN
 	1    5400 3750
@@
 F 0 "C2" H 3425 3450 50  0000 L CNN
 F 1 "4.7u" H 3425 3250 50  0000 L CNN
-F 2 "" H 3438 3200 50  0001 C CNN
+F 2 "Capacitors_SMD:C_0805_HandSoldering" H 3438 3200 50  0001 C CNN
 F 3 "" H 3400 3350 50  0000 C CNN
 	1    3400 3350
@@
 F 0 "R2" V 4380 2400 50  0000 C CNN
 F 1 "100k" V 4300 2400 50  0000 C CNN
-F 2 "" V 4230 2400 50  0001 C CNN
+F 2 "Resistors_SMD:R_0805_HandSoldering" V 4230 2400 50  0001 C CNN
 F 3 "" H 4300 2400 50  0000 C CNN
 	1    4300 2400
@@
 F 0 "R3" V 4580 2400 50  0000 C CNN
 F 1 "100k" V 4500 2400 50  0000 C CNN
-F 2 "" V 4430 2400 50  0001 C CNN
+F 2 "Resistors_SMD:R_0805_HandSoldering" V 4430 2400 50  0001 C CNN
 F 3 "" H 4500 2400 50  0000 C CNN
 	1    4500 2400
@@
 F 0 "J2" H 2750 4500 50  0000 C CNN
 F 1 "BATT_CONN" V 2850 4350 50  0000 C CNN
-F 2 "" H 2750 4350 50  0001 C CNN
+F 2 "Connectors_JST:JST_PH_S2B-PH-K_02x2.00mm_Angled" H 2750 4350 50  0001 C CNN
 F 3 "" H 2750 4350 50  0001 C CNN
 	1    2750 4350

Commit message: easier power mgmt
use MAX1811 chip
Parts:
- removed R3: 100k, Resistors_SMD:R_0805_HandSoldering, symbol R
- removed R4, R5: 1k, Resistors_SMD:R_0805_HandSoldering, symbol R
- removed R6: 10k, Resistors_SMD:R_0805_HandSoldering, symbol R
- removed U3: BQ24075, Housings_DFN_QFN:QFN-16-1EP_3x3mm_Pitch0.5mm, symbol BQ24075
- added U3: MAX1811, Housings_SOIC:SOIC-8_3.9x4.9mm_Pitch1.27mm, symbol MAX1811
- P1: symbol USB_OTG -> USB_OTG-RESCUE-soilsensor
- R2: value 100k -> 10k
Connections:
- net labels added: EN
- net labels removed: ~PGOOD
- wire segments 47 -> 30
- no-connect marks 5 -> 4
Other:
- moved on the sheet: C2, C3, J2

Commit message: update sensor
Parts:
- R2: footprint Resistors_SMD:R_0805_HandSoldering -> Resistors_SMD:R_0603_HandSoldering
Changed lines of the file:
@@
 $EndComp
 $Comp
-L GND #PWR09
+L GND #PWR010
 U 1 1 59568C2C
 P 6100 3600
-F 0 "#PWR09" H 6100 3350 50  0001 C CNN
+F 0 "#PWR010" H 6100 3350 50  0001 C CNN
 F 1 "GND" H 6100 3450 50  0000 C CNN
 F 2 "" H 6100 3600 50  0000 C CNN
@@
 $EndComp
 $Comp
-L VDD #PWR010
+L VDD #PWR011
 U 1 1 59568C2F
 P 6500 2750
-F 0 "#PWR010" H 6500 2600 50  0001 C CNN
+F 0 "#PWR011" H 6500 2600 50  0001 C CNN
 F 1 "VDD" H 6500 2900 50  0000 C CNN
 F 2 "" H 6500 2750 50  0000 C CNN
@@
 $EndComp
 $Comp
-L GND #PWR011
+L GND #PWR012
 U 1 1 59568C34
 P 3400 3850
-F 0 "#PWR011" H 3400 3600 50  0001 C CNN
+F 0 "#PWR012" H 3400 3600 50  0001 C CNN
 F 1 "GND" H 3400 3700 50  0000 C CNN
 F 2 "" H 3400 3850 50  0000 C CNN
@@
 $EndComp
 $Comp
-L GND #PWR012
+L GND #PWR013
 U 1 1 59568C3A
 P 3700 5250
-F 0 "#PWR012" H 3700 5000 50  0001 C CNN
+F 0 "#PWR013" H 3700 5000 50  0001 C CNN
 F 1 "GND" H 3700 5100 50  0000 C CNN
 F 2 "" H 3700 5250 50  0000 C CNN
@@
 $EndComp
 $Comp
-L +BATT #PWR013
+L +BATT #PWR014
 U 1 1 59568C5B
 P 3700 4750
-F 0 "#PWR013" H 3700 4600 50  0001 C CNN
+F 0 "#PWR014" H 3700 4600 50  0001 C CNN
 F 1 "+BATT" H 3700 4890 50  0000 C CNN
 F 2 "" H 3700 4750 50  0000 C CNN
@@
 Connection ~ 4350 3750
 $Comp
-L +BATT #PWR014
+L +BATT #PWR015
 U 1 1 5979B653
 P 5000 3000
-F 0 "#PWR014" H 5000 2850 50  0001 C CNN
+F 0 "#PWR015" H 5000 2850 50  0001 C CNN
 F 1 "+BATT" H 5000 3140 50  0000 C CNN
 F 2 "" H 5000 3000 50  0000 C CNN
@@
 	5700 2950 5800 2950
 $Comp
-L +BATT #PWR015
+L +BATT #PWR016
 U 1 1 5979B728
 P 5700 2800
-F 0 "#PWR015" H 5700 2650 50  0001 C CNN
+F 0 "#PWR016" H 5700 2650 50  0001 C CNN
 F 1 "+BATT" H 5700 2940 50  0000 C CNN
 F 2 "" H 5700 2800 50  0000 C CNN
@@
 F 0 "R2" V 3930 3000 50  0000 C CNN
 F 1 "10k" V 3850 3000 50  0000 C CNN
-F 2 "Resistors_SMD:R_0805_HandSoldering" V 3780 3000 50  0001 C CNN
+F 2 "Resistors_SMD:R_0603_HandSoldering" V 3780 3000 50  0001 C CNN
 F 3 "" H 3850 3000 50  0001 C CNN
 	1    3850 3000

Commit message: improve power mgmt schematics
Parts:
- removed U3: MAX1811, Housings_SOIC:SOIC-8_3.9x4.9mm_Pitch1.27mm, symbol MAX1811
- removed U4: MCP1700-3002E_SOT23, TO_SOT_Packages_SMD:SOT-23, symbol MCP1700-3002E_SOT23
- added D2: BAT20J, Diodes_SMD:SOD-323, symbol D_Schottky
- added Q1: Q_NMOS_DGS, TO_SOT_Packages_SMD:SOT-23, symbol Q_NMOS_DGS
- added Q2: Q_PMOS_DGS, TO_SOT_Packages_SMD:SOT-23, symbol Q_PMOS_DGS
- added R7: 8.2k, Resistors_SMD:R_0603, symbol R
- added R8: 10k, Resistors_SMD:R_0603, symbol R
- added U3: MCP73811T, TO_SOT_Packages_SMD:SOT-23-5, symbol MCP73812T-420I/OT
- added U4: AP2204K-3.0, TO_SOT_Packages_SMD:SOT-23-5, symbol AP2204K-3.0
- C2, C4: footprint Capacitors_SMD:C_0805_HandSoldering -> Capacitors_SMD:C_0805
- C3: value 22u -> 4.7u; footprint Capacitors_SMD:C_0805_HandSoldering -> Capacitors_SMD:C_0805
- C5: value 1u -> 2.2u; footprint Capacitors_SMD:C_0805_HandSoldering -> Capacitors_SMD:C_0805
- R2: value 10k -> 3.3k; footprint Resistors_SMD:R_0603_HandSoldering -> Resistors_SMD:R_0603
Connections:
- net labels added: BATT_V, BATT_V_EN
- net labels removed: EN, ~CHG
- wire segments 30 -> 40
- no-connect marks 4 -> 0
Other:
- moved on the sheet: C3, C4, C5, P1

Commit message: fix power mgmt
Parts:
- C2, C3, C4, C5: footprint Capacitors_SMD:C_0805 -> Capacitors_SMD:C_0603
Connections:
- wire segments 40 -> 42
Changed lines of the file:
@@
 LIBS:rfcom
 LIBS:maxim
-LIBS:battery_management
+LIBS:sensors
+LIBS:Battery_Management
 LIBS:soilsensor-cache
 EELAYER 25 0
@@
 F 0 "C4" H 6075 3450 50  0000 L CNN
 F 1 "1u" H 6075 3250 50  0000 L CNN
-F 2 "Capacitors_SMD:C_0805" H 6088 3200 50  0001 C CNN
+F 2 "Capacitors_SMD:C_0603" H 6088 3200 50  0001 C CNN
 F 3 "" H 6050 3350 50  0000 C CNN
 	1    6050 3350
@@
 F 0 "C5" H 7125 3450 50  0000 L CNN
 F 1 "2.2u" H 7125 3250 50  0000 L CNN
-F 2 "Capacitors_SMD:C_0805" H 7138 3200 50  0001 C CNN
+F 2 "Capacitors_SMD:C_0603" H 7138 3200 50  0001 C CNN
 F 3 "" H 7100 3350 50  0000 C CNN
 	1    7100 3350
@@
 $EndComp
 $Comp
-L GND #PWR010
+L GND #PWR08
 U 1 1 59568C2C
 P 6700 3750
-F 0 "#PWR010" H 6700 3500 50  0001 C CNN
+F 0 "#PWR08" H 6700 3500 50  0001 C CNN
 F 1 "GND" H 6700 3600 50  0000 C CNN
 F 2 "" H 6700 3750 50  0000 C CNN
@@
 $EndComp
 $Comp
-L VDD #PWR011
+L VDD #PWR09
 U 1 1 59568C2F
 P 7100 2900
-F 0 "#PWR011" H 7100 2750 50  0001 C CNN
+F 0 "#PWR09" H 7100 2750 50  0001 C CNN
 F 1 "VDD" H 7100 3050 50  0000 C CNN
 F 2 "" H 7100 2900 50  0000 C CNN
@@
 F 0 "C3" H 4775 3300 50  0000 L CNN
 F 1 "4.7u" H 4775 3100 50  0000 L CNN
-F 2 "Capacitors_SMD:C_0805" H 4788 3050 50  0001 C CNN
+F 2 "Capacitors_SMD:C_0603" H 4788 3050 50  0001 C CNN
 F 3 "" H 4750 3200 50  0000 C CNN
 	1    4750 3200
@@
 $EndComp
 $Comp
-L GND #PWR012
+L GND #PWR010
 U 1 1 59568C3A
 P 3500 5100
-F 0 "#PWR012" H 3500 4850 50  0001 C CNN
+F 0 "#PWR010" H 3500 4850 50  0001 C CNN
 F 1 "GND" H 3500 4950 50  0000 C CNN
 F 2 "" H 3500 5100 50  0000 C CNN
@@
 $EndComp
 $Comp
-L +BATT #PWR013
+L +BATT #PWR011
 U 1 1 59568C5B
 P 3500 4900
-F 0 "#PWR013" H 3500 4750 50  0001 C CNN
+F 0 "#PWR011" H 3500 4750 50  0001 C CNN
 F 1 "+BATT" H 3500 5040 50  0000 C CNN
 F 2 "" H 3500 4900 50  0000 C CNN
@@
 Connection ~ 6700 3650
 $Comp
-L +BATT #PWR014
+L +BATT #PWR012
 U 1 1 5979B653
 P 4750 2900
-F 0 "#PWR014" H 4750 2750 50  0001 C CNN
+F 0 "#PWR012" H 4750 2750 50  0001 C CNN
 F 1 "+BATT" H 4750 3040 50  0000 C CNN
 F 2 "" H 4750 2900 50  0000 C CNN
@@
 	3450 3200 3550 3200
 $Comp
-L GND #PWR015
+L GND #PWR013
 U 1 1 59D3742E
 P 2650 3750
-F 0 "#PWR015" H 2650 3500 50  0001 C CNN
+F 0 "#PWR013" H 2650 3500 50  0001 C CNN
 F 1 "GND" H 2650 3600 50  0000 C CNN
 F 2 "" H 2650 3750 50  0000 C CNN
@@
 $EndComp
 $Comp
-L GND #PWR016
+L GND #PWR014
 U 1 1 59D37473
 P 4750 3450
-F 0 "#PWR016" H 4750 3200 50  0001 C CNN
+F 0 "#PWR014" H 4750 3200 50  0001 C CNN
 F 1 "GND" H 4750 3300 50  0000 C CNN
 F 2 "" H 4750 3450 50  0000 C CNN
@@
 F 0 "C2" H 3175 3400 50  0000 L CNN
 F 1 "4.7u" H 3175 3200 50  0000 L CNN
-F 2 "Capacitors_SMD:C_0805" H 3188 3150 50  0001 C CNN
+F 2 "Capacitors_SMD:C_0603" H 3188 3150 50  0001 C CNN
 F 3 "" H 3150 3300 50  0000 C CNN
 	1    3150 3300
@@
 $EndComp
 $Comp
-L GND #PWR017
+L GND #PWR015
 U 1 1 59D39161
 P 5050 2750
-F 0 "#PWR017" H 5050 2500 50  0001 C CNN
+F 0 "#PWR015" H 5050 2500 50  0001 C CNN
 F 1 "GND" H 5050 2600 50  0000 C CNN
 F 2 "" H 5050 2750 50  0000 C CNN
@@
 $EndComp
 $Comp
-L GND #PWR018
+L GND #PWR016
 U 1 1 59D397E4
 P 4750 5550
-F 0 "#PWR018" H 4750 5300 50  0001 C CNN
+F 0 "#PWR016" H 4750 5300 50  0001 C CNN
 F 1 "GND" H 4750 5400 50  0000 C CNN
 F 2 "" H 4750 5550 50  0000 C CNN
@@
 $EndComp
 $Comp
-L +BATT #PWR019
+L +BATT #PWR017
 U 1 1 59D39851
 P 4750 4150
-F 0 "#PWR019" H 4750 4000 50  0001 C CNN
+F 0 "#PWR017" H 4750 4000 50  0001 C CNN
 F 1 "+BATT" H 4750 4290 50  0000 C CNN
 F 2 "" H 4750 4150 50  0000 C CNN
@@
 Text HLabel 4450 5250 0    60   Input ~ 0
 BATT_V_EN
+Wire Wire Line
+	6400 3100 6250 3100
+Wire Wire Line
+	6250 3100 6250 3000
+Connection ~ 6250 3000
 $EndSCHEMATC

Commit message: change mosfet layouts
Parts:
- removed Q1: Q_NMOS_DGS, TO_SOT_Packages_SMD:SOT-23, symbol Q_NMOS_DGS
- removed Q2: Q_PMOS_DGS, TO_SOT_Packages_SMD:SOT-23, symbol Q_PMOS_DGS
- added Q?: Q_NMOS_GSD, symbol Q_NMOS_GSD
- added Q?: Q_PMOS_GSD, symbol Q_PMOS_GSD
Changed lines of the file:
@@
 Wire Wire Line
 	6050 3000 6050 3200
-$Comp
-L Q_PMOS_DGS Q2
-U 1 1 59D38FB3
-P 5500 2900
-F 0 "Q2" H 5700 2950 50  0000 L CNN
-F 1 "Q_PMOS_DGS" H 5700 2850 50  0000 L CNN
-F 2 "TO_SOT_Packages_SMD:SOT-23" H 5700 3000 50  0001 C CNN
-F 3 "" H 5500 2900 50  0001 C CNN
-	1    5500 2900
-	0    -1   1    0
-$EndComp
 Connection ~ 6050 3000
 $Comp
@@
 Wire Wire Line
 	5500 2400 3450 2400
-$Comp
-L Q_NMOS_DGS Q1
-U 1 1 59D395F8
-P 4650 5250
-F 0 "Q1" H 4850 5300 50  0000 L CNN
-F 1 "Q_NMOS_DGS" H 4850 5200 50  0000 L CNN
-F 2 "TO_SOT_Packages_SMD:SOT-23" H 4850 5350 50  0001 C CNN
-F 3 "" H 4650 5250 50  0001 C CNN
-	1    4650 5250
-	1    0    0    -1
-$EndComp
 $Comp
 L R R2
@@
 	6250 3100 6250 3000
 Connection ~ 6250 3000
+$Comp
+L Q_NMOS_GSD Q?
+U 1 1 59E474DA
+P 4650 5250
+F 0 "Q?" H 4850 5300 50  0000 L CNN
+F 1 "Q_NMOS_GSD" H 4850 5200 50  0000 L CNN
+F 2 "" H 4850 5350 50  0001 C CNN
+F 3 "" H 4650 5250 50  0001 C CNN
+	1    4650 5250
+	1    0    0    -1
+$EndComp
+$Comp
+L Q_PMOS_GSD Q?
+U 1 1 59E47873
+P 5500 2900
+F 0 "Q?" H 5700 2950 50  0000 L CNN
+F 1 "Q_PMOS_GSD" H 5700 2850 50  0000 L CNN
+F 2 "" H 5700 3000 50  0001 C CNN
+F 3 "" H 5500 2900 50  0001 C CNN
+	1    5500 2900
+	0    -1   1    0
+$EndComp
 $EndSCHEMATC
