File: PowerMgmt.sch (KiCad schematic (older format))
At the start: 14 parts, among them J2 BATT_CONN, P1 USB_OTG, Q1 Q_NMOS_GSD, Q2 Q_PMOS_GSD, U3 MCP73811T, U4 AP2204K-3.0

Commit message: update power mgmt
Parts:
- P1: footprint Connect:USB_Micro-B -> Connectors_USB:USB_Micro-B_Molex_47346-0001
Connections:
- net VBUS: now reaches C4.1, D2.1 (K), Q2.2 (S), U4.1 (VIN), U4.3 (EN)
Changed lines of the file:
@@
 F 0 "P1" H 2750 2850 50  0000 C CNN
 F 1 "USB_OTG" H 2650 3550 50  0000 C CNN
-F 2 "Connect:USB_Micro-B" V 2600 3100 50  0001 C CNN
+F 2 "Connectors_USB:USB_Micro-B_Molex_47346-0001" V 2600 3100 50  0001 C CNN
 F 3 "" V 2600 3100 50  0000 C CNN
 	1    2650 3200
@@
 BATT_V_EN
 Wire Wire Line
-	6400 3100 6250 3100
-Wire Wire Line
-	6250 3100 6250 3000
+	6250 3100 6400 3100
+Wire Wire Line
+	6250 2850 6250 3100
 Connection ~ 6250 3000
 $Comp
@@
 	0    -1   1    0
 $EndComp
+$Comp
+L VBUS #PWR?
+U 1 1 59F888BF
+P 6250 2850
+F 0 "#PWR?" H 6250 2700 50  0001 C CNN
+F 1 "VBUS" H 6250 3000 50  0000 C CNN
+F 2 "" H 6250 2850 50  0001 C CNN
+F 3 "" H 6250 2850 50  0001 C CNN
+	1    6250 2850
+	1    0    0    -1
+$EndComp
 $EndSCHEMATC

Commit message: update schematics
Parts:
- added R10: 1.8k, Resistors_SMD:R_0603, symbol R
- R2: value 3.3k -> 1.5k
Connections:
- net BATT_V: now also R10.2; no longer R2.2
- new net: R10.1, R2.2
- no-connect marks 0 -> 1
Other:
- moved on the sheet: R2
Changed lines of the file:
@@
 L R R2
 U 1 1 59D3966F
-P 4750 4400
-F 0 "R2" V 4830 4400 50  0000 C CNN
-F 1 "3.3k" V 4750 4400 50  0000 C CNN
-F 2 "Resistors_SMD:R_0603" V 4680 4400 50  0001 C CNN
-F 3 "" H 4750 4400 50  0001 C CNN
-	1    4750 4400
+P 4750 4000
+F 0 "R2" V 4830 4000 50  0000 C CNN
+F 1 "1.5k" V 4750 4000 50  0000 C CNN
+F 2 "Resistors_SMD:R_0603" V 4680 4000 50  0001 C CNN
+F 3 "" H 4750 4000 50  0001 C CNN
+	1    4750 4000
 	1    0    0    -1
 $EndComp
@@
 L +BATT #PWR017
 U 1 1 59D39851
-P 4750 4150
-F 0 "#PWR017" H 4750 4000 50  0001 C CNN
-F 1 "+BATT" H 4750 4290 50  0000 C CNN
-F 2 "" H 4750 4150 50  0000 C CNN
-F 3 "" H 4750 4150 50  0000 C CNN
-	1    4750 4150
+P 4750 3850
+F 0 "#PWR017" H 4750 3700 50  0001 C CNN
+F 1 "+BATT" H 4750 3990 50  0000 C CNN
+F 2 "" H 4750 3850 50  0000 C CNN
+F 3 "" H 4750 3850 50  0000 C CNN
+	1    4750 3850
 	1    0    0    -1
 $EndComp
@@
 $EndComp
 $Comp
-L VBUS #PWR?
+L VBUS #PWR018
 U 1 1 59F888BF
 P 6250 2850
-F 0 "#PWR?" H 6250 2700 50  0001 C CNN
+F 0 "#PWR018" H 6250 2700 50  0001 C CNN
 F 1 "VBUS" H 6250 3000 50  0000 C CNN
 F 2 "" H 6250 2850 50  0001 C CNN
@@
 	1    0    0    -1
 $EndComp
+NoConn ~ 2550 3600
+$Comp
+L R R10
+U 1 1 5A01AE6C
+P 4750 4400
+F 0 "R10" V 4830 4400 50  0000 C CNN
+F 1 "1.8k" V 4750 4400 50  0000 C CNN
+F 2 "Resistors_SMD:R_0603" V 4680 4400 50  0001 C CNN
+F 3 "" H 4750 4400 50  0001 C CNN
+	1    4750 4400
+	1    0    0    -1
+$EndComp
