File: soilsensor.sch (KiCad schematic (older format))
At the start: 5 parts

Commit message: fix minors, make annotations
Parts:
- U1: renamed from U?; footprint (none) -> TO_SOT_Packages_THT:TO-92_Inline_Narrow_Oval
- U2: renamed from U?; footprint (none) -> kicad-RF_Modules:RFDigital_RFD77101
- gave numbers to parts that had none: 3
Changed lines of the file:
@@
 $EndDescr
 $Comp
-L RFD77101 U?
+L RFD77101 U2
 U 1 1 595643C3
 P 6400 3400
-F 0 "U?" H 6200 4800 50  0000 C CNN
+F 0 "U2" H 6200 4800 50  0000 C CNN
 F 1 "RFD77101" H 6100 4700 50  0000 C CNN
-F 2 "" H 7200 2200 50  0001 C CNN
+F 2 "kicad-RF_Modules:RFDigital_RFD77101" H 7200 2200 50  0001 C CNN
 F 3 "" H 6400 1900 50  0001 C CNN
 	1    6400 3400
@@
 $EndSheet
 $Comp
-L C C?
+L C C1
 U 1 1 59567DAD
 P 5300 1800
-F 0 "C?" H 5325 1900 50  0000 L CNN
+F 0 "C1" H 5325 1900 50  0000 L CNN
 F 1 "1u" H 5325 1700 50  0000 L CNN
 F 2 "" H 5338 1650 50  0001 C CNN
@@
 $EndComp
 $Comp
-L GND #PWR?
+L GND #PWR01
 U 1 1 59567E26
 P 6100 4800
-F 0 "#PWR?" H 6100 4550 50  0001 C CNN
+F 0 "#PWR01" H 6100 4550 50  0001 C CNN
 F 1 "GND" H 6100 4650 50  0000 C CNN
 F 2 "" H 6100 4800 50  0001 C CNN
@@
 	6100 4700 6100 4800
 $Comp
-L GND #PWR?
+L GND #PWR02
 U 1 1 59567F28
 P 5300 2050
-F 0 "#PWR?" H 5300 1800 50  0001 C CNN
+F 0 "#PWR02" H 5300 1800 50  0001 C CNN
 F 1 "GND" H 5300 1900 50  0000 C CNN
 F 2 "" H 5300 2050 50  0001 C CNN
@@
 $EndComp
 $Comp
-L VDD #PWR?
+L VDD #PWR03
 U 1 1 59567FFA
 P 5300 1550
-F 0 "#PWR?" H 5300 1400 50  0001 C CNN
+F 0 "#PWR03" H 5300 1400 50  0001 C CNN
 F 1 "VDD" H 5300 1700 50  0000 C CNN
 F 2 "" H 5300 1550 50  0001 C CNN
@@
 	5700 3000 4500 3000
 $Comp
-L CONN_01X06 J?
+L CONN_01X06 J1
 U 1 1 595676C1
 P 4000 1900
-F 0 "J?" H 4000 2250 50  0000 C CNN
+F 0 "J1" H 4000 2250 50  0000 C CNN
 F 1 "CONN_01X06" V 4100 1900 50  0000 C CNN
 F 2 "" H 4000 1900 50  0001 C CNN
@@
 $EndComp
 $Comp
-L VDD #PWR?
+L VDD #PWR04
 U 1 1 5956777F
 P 4300 1600
-F 0 "#PWR?" H 4300 1450 50  0001 C CNN
+F 0 "#PWR04" H 4300 1450 50  0001 C CNN
 F 1 "VDD" H 4300 1750 50  0000 C CNN
 F 2 "" H 4300 1600 50  0001 C CNN
@@
 $EndComp
 $Comp
-L GND #PWR?
+L GND #PWR05
 U 1 1 595677AB
 P 4300 2200
-F 0 "#PWR?" H 4300 1950 50  0001 C CNN
+F 0 "#PWR05" H 4300 1950 50  0001 C CNN
 F 1 "GND" H 4300 2050 50  0000 C CNN
 F 2 "" H 4300 2200 50  0001 C CNN
@@
 GPIO1
 $Comp
-L DS18B20 U?
+L DS18B20 U1
 U 1 1 59567BCA
 P 3950 4050
-F 0 "U?" H 3800 4300 50  0000 C CNN
+F 0 "U1" H 3800 4300 50  0000 C CNN
 F 1 "DS18B20" H 3950 3800 50  0000 C CNN
-F 2 "" H 3800 4300 50  0001 C CNN
+F 2 "TO_SOT_Packages_THT:TO-92_Inline_Narrow_Oval" H 3800 4300 50  0001 C CNN
 F 3 "" H 3800 4300 50  0001 C CNN
 	1    3950 4050
@@
 $EndComp
 $Comp
-L R R?
+L R R1
 U 1 1 59567D40
 P 4600 3800
-F 0 "R?" V 4680 3800 50  0000 C CNN
+F 0 "R1" V 4680 3800 50  0000 C CNN
 F 1 "4.7k" V 4600 3800 50  0000 C CNN
 F 2 "" V 4530 3800 50  0001 C CNN
@@
 $EndComp
 $Comp
-L GND #PWR?
+L GND #PWR06
 U 1 1 59567F04
 P 4300 4250
-F 0 "#PWR?" H 4300 4000 50  0001 C CNN
+F 0 "#PWR06" H 4300 4000 50  0001 C CNN
 F 1 "GND" H 4300 4100 50  0000 C CNN
 F 2 "" H 4300 4250 50  0001 C CNN
@@
 Connection ~ 4300 4150
 $Comp
-L VDD #PWR?
+L VDD #PWR07
 U 1 1 59568035
 P 4600 3550
-F 0 "#PWR?" H 4600 3400 50  0001 C CNN
+F 0 "#PWR07" H 4600 3400 50  0001 C CNN
 F 1 "VDD" H 4600 3700 50  0000 C CNN
 F 2 "" H 4600 3550 50  0001 C CNN
