File: soilsensor.sch (KiCad schematic (older format))
At the start: 5 parts, among them J1 CONN_01X06, U1 DS18B20, U2 RFD77101

Commit message: update footprints
Parts:
- C1: footprint (none) -> Capacitors_SMD:C_0805_HandSoldering
- J1: footprint (none) -> Socket_Strips:Socket_Strip_Straight_1x06
- R1: footprint (none) -> Resistors_SMD:R_0805_HandSoldering
Changed lines of the file:
@@
 F 0 "C1" H 5325 1900 50  0000 L CNN
 F 1 "1u" H 5325 1700 50  0000 L CNN
-F 2 "" H 5338 1650 50  0001 C CNN
+F 2 "Capacitors_SMD:C_0805_HandSoldering" H 5338 1650 50  0001 C CNN
 F 3 "" H 5300 1800 50  0001 C CNN
 	1    5300 1800
@@
 F 0 "J1" H 4000 2250 50  0000 C CNN
 F 1 "CONN_01X06" V 4100 1900 50  0000 C CNN
-F 2 "" H 4000 1900 50  0001 C CNN
+F 2 "Socket_Strips:Socket_Strip_Straight_1x06" H 4000 1900 50  0001 C CNN
 F 3 "" H 4000 1900 50  0001 C CNN
 	1    4000 1900
@@
 F 0 "R1" V 4680 3800 50  0000 C CNN
 F 1 "4.7k" V 4600 3800 50  0000 C CNN
-F 2 "" V 4530 3800 50  0001 C CNN
+F 2 "Resistors_SMD:R_0805_HandSoldering" V 4530 3800 50  0001 C CNN
 F 3 "" H 4600 3800 50  0001 C CNN
 	1    4600 3800

Commit message: finish pcb
Connections:
- wire segments 21 -> 27
- no-connect marks 5 -> 0
Changed lines of the file:
@@
 $EndSheet
 $Sheet
-S 3700 2900 800  200
+S 4100 2950 800  200
 U 59567161
 F0 "CapacitiveSoilSensor" 60
 F1 "CapacitiveSoilSensor.sch" 60
-F2 "SensorOut" I R 4500 3000 60
+F2 "SensorOut" I R 4900 3050 60
 $EndSheet
 $Comp
@@
 $EndComp
 Wire Wire Line
-	5900 4700 6300 4700
+	5900 4700 6800 4700
 Connection ~ 6000 4700
 Connection ~ 6100 4700
@@
 	6400 1600 6400 2100
 Connection ~ 5300 1600
-NoConn ~ 6700 4700
-NoConn ~ 6800 4700
-NoConn ~ 6500 4700
-NoConn ~ 6600 4700
-NoConn ~ 6400 4700
 Wire Wire Line
 	7100 2500 7500 2500
 Wire Wire Line
 	7100 2600 7500 2600
-Wire Wire Line
-	5700 3000 4500 3000
 $Comp
 L CONN_01X06 J1
@@
 	5350 3500 5700 3500
 Connection ~ 4600 4050
+Wire Wire Line
+	4900 3050 5550 3050
+Wire Wire Line
+	5550 3050 5550 3200
+Wire Wire Line
+	5550 3200 5700 3200
+$Comp
+L VDD #PWR?
+U 1 1 596CB151
+P 8800 2650
+F 0 "#PWR?" H 8800 2500 50  0001 C CNN
+F 1 "VDD" H 8800 2800 50  0000 C CNN
+F 2 "" H 8800 2650 50  0001 C CNN
+F 3 "" H 8800 2650 50  0001 C CNN
+	1    8800 2650
+	1    0    0    -1
+$EndComp
+Wire Wire Line
+	7100 2700 7400 2700
+Wire Wire Line
+	7400 2700 7400 2850
+Wire Wire Line
+	7400 2850 8800 2850
+Wire Wire Line
+	8800 2850 8800 2650
+Connection ~ 6300 4700
+Connection ~ 6400 4700
+Connection ~ 6500 4700
+Connection ~ 6600 4700
+Connection ~ 6700 4700
 $EndSCHEMATC

Commit message: a lot of fixes, finished one-sided layout
Changed lines of the file:
@@
 EESchema Schematic File Version 2
+LIBS:soilsensor-rescue
 LIBS:power
 LIBS:device
@@
 $EndComp
 $Sheet
-S 7500 2400 800  300
+S 7500 2500 800  300
 U 595666C6
 F0 "PowerMgmt" 60
 F1 "PowerMgmt.sch" 60
-F2 "~PGOOD" I L 7500 2500 60
-F3 "~CHG" I L 7500 2600 60
+F2 "~CHG" I L 7500 2600 60
+F3 "EN" I L 7500 2700 60
 $EndSheet
 $Sheet
@@
 	6400 1600 6400 2100
 Connection ~ 5300 1600
-Wire Wire Line
-	7100 2500 7500 2500
-Wire Wire Line
-	7100 2600 7500 2600
 $Comp
 L CONN_01X06 J1
@@
 	5550 3200 5700 3200
 $Comp
-L VDD #PWR?
+L VDD #PWR08
 U 1 1 596CB151
-P 8800 2650
-F 0 "#PWR?" H 8800 2500 50  0001 C CNN
-F 1 "VDD" H 8800 2800 50  0000 C CNN
-F 2 "" H 8800 2650 50  0001 C CNN
-F 3 "" H 8800 2650 50  0001 C CNN
-	1    8800 2650
-	1    0    0    -1
-$EndComp
-Wire Wire Line
-	7100 2700 7400 2700
-Wire Wire Line
-	7400 2700 7400 2850
-Wire Wire Line
-	7400 2850 8800 2850
-Wire Wire Line
-	8800 2850 8800 2650
+P 7300 2350
+F 0 "#PWR08" H 7300 2200 50  0001 C CNN
+F 1 "VDD" H 7300 2500 50  0000 C CNN
+F 2 "" H 7300 2350 50  0001 C CNN
+F 3 "" H 7300 2350 50  0001 C CNN
+	1    7300 2350
+	1    0    0    -1
+$EndComp
 Connection ~ 6300 4700
 Connection ~ 6400 4700
@@
 Connection ~ 6600 4700
 Connection ~ 6700 4700
+Wire Wire Line
+	7100 2600 7500 2600
+Wire Wire Line
+	7100 2700 7500 2700
+Wire Wire Line
+	7100 2500 7300 2500
+Wire Wire Line
+	7300 2500 7300 2350
+$Comp
+L GND #PWR?
+U 1 1 59807528
+P 7300 2900
+F 0 "#PWR?" H 7300 2650 50  0001 C CNN
+F 1 "GND" H 7300 2750 50  0000 C CNN
+F 2 "" H 7300 2900 50  0001 C CNN
+F 3 "" H 7300 2900 50  0001 C CNN
+	1    7300 2900
+	1    0    0    -1
+$EndComp
+Wire Wire Line
+	7100 2800 7300 2800
+Wire Wire Line
+	7300 2800 7300 2900
 $EndSCHEMATC

Commit message: update sensor
Parts:
- C1: footprint Capacitors_SMD:C_0805_HandSoldering -> Capacitors_SMD:C_1206_HandSoldering
- R1: footprint Resistors_SMD:R_0805_HandSoldering -> Resistors_SMD:R_0603_HandSoldering
Changed lines of the file:
@@
 F 0 "C1" H 5325 1900 50  0000 L CNN
 F 1 "1u" H 5325 1700 50  0000 L CNN
-F 2 "Capacitors_SMD:C_0805_HandSoldering" H 5338 1650 50  0001 C CNN
+F 2 "Capacitors_SMD:C_1206_HandSoldering" H 5338 1650 50  0001 C CNN
 F 3 "" H 5300 1800 50  0001 C CNN
 	1    5300 1800
@@
 Text Label 4200 1850 0    60   ~ 0
 SWDCLK
+Text Label 4200 2050 0    60   ~ 0
+GPIO0
 Text Label 4200 1950 0    60   ~ 0
-GPIO0
-Text Label 4200 2050 0    60   ~ 0
 GPIO1
 Text Label 5700 2500 2    60   ~ 0
@@
 F 0 "R1" V 4680 3800 50  0000 C CNN
 F 1 "4.7k" V 4600 3800 50  0000 C CNN
-F 2 "Resistors_SMD:R_0805_HandSoldering" V 4530 3800 50  0001 C CNN
+F 2 "Resistors_SMD:R_0603_HandSoldering" V 4530 3800 50  0001 C CNN
 F 3 "" H 4600 3800 50  0001 C CNN
 	1    4600 3800
@@
 	7300 2500 7300 2350
 $Comp
-L GND #PWR?
+L GND #PWR09
 U 1 1 59807528
 P 7300 2900
-F 0 "#PWR?" H 7300 2650 50  0001 C CNN
+F 0 "#PWR09" H 7300 2650 50  0001 C CNN
 F 1 "GND" H 7300 2750 50  0000 C CNN
 F 2 "" H 7300 2900 50  0001 C CNN

Commit message: update schematic for new components
Parts:
- removed J1: CONN_01X06, Socket_Strips:Socket_Strip_Straight_1x06, symbol CONN_01X06
- added J1: CONN_01X07, Pin_Headers:Pin_Header_Straight_1x07_Pitch2.54mm, symbol CONN_01X07
- C1: footprint Capacitors_SMD:C_1206_HandSoldering -> Capacitors_SMD:C_1206
- R1: footprint Resistors_SMD:R_0603_HandSoldering -> Resistors_SMD:R_0603
- U1: footprint TO_SOT_Packages_THT:TO-92_Inline_Narrow_Oval -> Housings_SSOP:MSOP-8_3x3mm_Pitch0.65mm
Connections:
- net labels added: V_BATT
- wire segments 27 -> 29
- no-connect marks 0 -> 1
Changed lines of the file:
@@
 $EndComp
 $Sheet
-S 7500 2500 800  300
+S 7700 2500 800  300
 U 595666C6
 F0 "PowerMgmt" 60
 F1 "PowerMgmt.sch" 60
-F2 "~CHG" I L 7500 2600 60
-F3 "EN" I L 7500 2700 60
+F2 "BATT_V" I L 7700 2700 60
+F3 "BATT_V_EN" I L 7700 2600 60
 $EndSheet
 $Sheet
-S 4100 2950 800  200
+S 4100 2950 800  300
 U 59567161
 F0 "CapacitiveSoilSensor" 60
 F1 "CapacitiveSoilSensor.sch" 60
 F2 "SensorOut" I R 4900 3050 60
+F3 "~EN" I R 4900 3150 60
 $EndSheet
 $Comp
@@
 F 0 "C1" H 5325 1900 50  0000 L CNN
 F 1 "1u" H 5325 1700 50  0000 L CNN
-F 2 "Capacitors_SMD:C_1206_HandSoldering" H 5338 1650 50  0001 C CNN
+F 2 "Capacitors_SMD:C_1206" H 5338 1650 50  0001 C CNN
 F 3 "" H 5300 1800 50  0001 C CNN
 	1    5300 1800
@@
 Connection ~ 5300 1600
 $Comp
-L CONN_01X06 J1
-U 1 1 595676C1
-P 4000 1900
-F 0 "J1" H 4000 2250 50  0000 C CNN
-F 1 "CONN_01X06" V 4100 1900 50  0000 C CNN
-F 2 "Socket_Strips:Socket_Strip_Straight_1x06" H 4000 1900 50  0001 C CNN
-F 3 "" H 4000 1900 50  0001 C CNN
-	1    4000 1900
-	-1   0    0    -1
-$EndComp
-$Comp
 L VDD #PWR04
 U 1 1 5956777F
-P 4300 1600
-F 0 "#PWR04" H 4300 1450 50  0001 C CNN
-F 1 "VDD" H 4300 1750 50  0000 C CNN
-F 2 "" H 4300 1600 50  0001 C CNN
-F 3 "" H 4300 1600 50  0001 C CNN
-	1    4300 1600
+P 4350 1750
+F 0 "#PWR04" H 4350 1600 50  0001 C CNN
+F 1 "VDD" H 4350 1900 50  0000 C CNN
+F 2 "" H 4350 1750 50  0001 C CNN
+F 3 "" H 4350 1750 50  0001 C CNN
+	1    4350 1750
 	1    0    0    -1
 $EndComp
@@
 L GND #PWR05
 U 1 1 595677AB
-P 4300 2200
-F 0 "#PWR05" H 4300 1950 50  0001 C CNN
-F 1 "GND" H 4300 2050 50  0000 C CNN
-F 2 "" H 4300 2200 50  0001 C CNN
-F 3 "" H 4300 2200 50  0001 C CNN
-	1    4300 2200
-	1    0    0    -1
-$EndComp
-Wire Wire Line
-	4200 2150 4300 2150
-Wire Wire Line
-	4300 2150 4300 2200
-Wire Wire Line
-	4200 1650 4300 1650
-Wire Wire Line
-	4300 1650 4300 1600
-Text Label 4200 1750 0    60   ~ 0
+P 3650 2050
+F 0 "#PWR05" H 3650 1800 50  0001 C CNN
+F 1 "GND" H 3650 1900 50  0000 C CNN
+F 2 "" H 3650 2050 50  0001 C CNN
+F 3 "" H 3650 2050 50  0001 C CNN
+	1    3650 2050
+	1    0    0    -1
+$EndComp
+Text Label 3600 1700 0    60   ~ 0
 SWDIO/RESET
-Text Label 4200 1850 0    60   ~ 0
+Text Label 3600 1600 0    60   ~ 0
 SWDCLK
-Text Label 4200 2050 0    60   ~ 0
+Text Label 3600 1500 0    60   ~ 0
 GPIO0
-Text Label 4200 1950 0    60   ~ 0
+Text Label 3600 1400 0    60   ~ 0
 GPIO1
 Text Label 5700 2500 2    60   ~ 0
@@
 F 0 "U1" H 3800 4300 50  0000 C CNN
 F 1 "DS18B20" H 3950 3800 50  0000 C CNN
-F 2 "TO_SOT_Packages_THT:TO-92_Inline_Narrow_Oval" H 3800 4300 50  0001 C CNN
+F 2 "Housings_SSOP:MSOP-8_3x3mm_Pitch0.65mm" H 3800 4300 50  0001 C CNN
 F 3 "" H 3800 4300 50  0001 C CNN
 	1    3950 4050
@@
 F 0 "R1" V 4680 3800 50  0000 C CNN
 F 1 "4.7k" V 4600 3800 50  0000 C CNN
-F 2 "Resistors_SMD:R_0603_HandSoldering" V 4530 3800 50  0001 C CNN
+F 2 "Resistors_SMD:R_0603" V 4530 3800 50  0001 C CNN
 F 3 "" H 4600 3800 50  0001 C CNN
 	1    4600 3800
@@
 Connection ~ 6700 4700
 Wire Wire Line
-	7100 2600 7500 2600
-Wire Wire Line
-	7100 2700 7500 2700
+	7100 2600 7700 2600
 Wire Wire Line
 	7100 2500 7300 2500
@@
 Wire Wire Line
 	7300 2800 7300 2900
+$Comp
+L CONN_01X07 J1
+U 1 1 59A3EC25
+P 3400 1700
+F 0 "J1" H 3400 2100 50  0000 C CNN
+F 1 "CONN_01X07" V 3500 1700 50  0000 C CNN
+F 2 "Pin_Headers:Pin_Header_Straight_1x07_Pitch2.54mm" H 3400 1700 50  0001 C CNN
+F 3 "" H 3400 1700 50  0001 C CNN
+	1    3400 1700
+	-1   0    0    1
+$EndComp
+Wire Wire Line
+	3600 2000 3650 2000
+Wire Wire Line
+	3650 2000 3650 2050
+Wire Wire Line
+	3600 1800 4350 1800
+Wire Wire Line
+	4350 1800 4350 1750
+NoConn ~ 3600 1900
+Text Label 7700 2700 2    60   ~ 0
+V_BATT
+Text Label 5700 3000 2    60   ~ 0
+V_BATT
+Wire Wire Line
+	4900 3150 5450 3150
+Wire Wire Line
+	5450 3150 5450 3600
+Wire Wire Line
+	5450 3600 5700 3600
 $EndSCHEMATC

Commit message: minors in schematic
rewiring etc.
Parts:
- removed U1: DS18B20, Housings_SSOP:MSOP-8_3x3mm_Pitch0.65mm, symbol DS18B20
- added U1: DS18B20U, Housings_SSOP:MSOP-8_3x3mm_Pitch0.65mm, symbol DS18B20U
- C1: footprint Capacitors_SMD:C_1206 -> Capacitors_SMD:C_0603
Connections:
- net labels added: SS_OUT, V_BATT_EN, ~SS_EN
- wire segments 29 -> 20
Changed lines of the file:
@@
 LIBS:rfcom
 LIBS:maxim
-LIBS:battery_management
+LIBS:sensors
+LIBS:Battery_Management
 LIBS:soilsensor-cache
 EELAYER 25 0
@@
 F 0 "C1" H 5325 1900 50  0000 L CNN
 F 1 "1u" H 5325 1700 50  0000 L CNN
-F 2 "Capacitors_SMD:C_1206" H 5338 1650 50  0001 C CNN
+F 2 "Capacitors_SMD:C_0603" H 5338 1650 50  0001 C CNN
 F 3 "" H 5300 1800 50  0001 C CNN
 	1    5300 1800
@@
 GPIO1
 $Comp
-L DS18B20 U1
-U 1 1 59567BCA
-P 3950 4050
-F 0 "U1" H 3800 4300 50  0000 C CNN
-F 1 "DS18B20" H 3950 3800 50  0000 C CNN
-F 2 "Housings_SSOP:MSOP-8_3x3mm_Pitch0.65mm" H 3800 4300 50  0001 C CNN
-F 3 "" H 3800 4300 50  0001 C CNN
-	1    3950 4050
-	-1   0    0    -1
-$EndComp
-$Comp
 L R R1
 U 1 1 59567D40
@@
 L GND #PWR06
 U 1 1 59567F04
-P 4300 4250
-F 0 "#PWR06" H 4300 4000 50  0001 C CNN
-F 1 "GND" H 4300 4100 50  0000 C CNN
-F 2 "" H 4300 4250 50  0001 C CNN
-F 3 "" H 4300 4250 50  0001 C CNN
-	1    4300 4250
+P 3950 4450
+F 0 "#PWR06" H 3950 4200 50  0001 C CNN
+F 1 "GND" H 3950 4300 50  0000 C CNN
+F 2 "" H 3950 4450 50  0001 C CNN
+F 3 "" H 3950 4450 50  0001 C CNN
+	1    3950 4450
 	-1   0    0    -1
 $EndComp
 Wire Wire Line
-	4250 4150 4300 4150
-Wire Wire Line
-	4300 3950 4300 4250
-Wire Wire Line
-	4250 4050 5350 4050
-Wire Wire Line
-	4250 3950 4300 3950
-Connection ~ 4300 4150
+	4250 4050 5150 4050
 $Comp
 L VDD #PWR07
@@
 	4600 3950 4600 4050
 Wire Wire Line
-	5350 4050 5350 3500
-Wire Wire Line
-	5350 3500 5700 3500
+	5150 4050 5150 3500
+Wire Wire Line
+	5150 3500 5700 3500
 Connection ~ 4600 4050
-Wire Wire Line
-	4900 3050 5550 3050
-Wire Wire Line
-	5550 3050 5550 3200
-Wire Wire Line
-	5550 3200 5700 3200
-$Comp
-L VDD #PWR08
-U 1 1 596CB151
-P 7300 2350
-F 0 "#PWR08" H 7300 2200 50  0001 C CNN
-F 1 "VDD" H 7300 2500 50  0000 C CNN
-F 2 "" H 7300 2350 50  0001 C CNN
-F 3 "" H 7300 2350 50  0001 C CNN
-	1    7300 2350
-	1    0    0    -1
-$EndComp
 Connection ~ 6300 4700
 Connection ~ 6400 4700
@@
 Connection ~ 6600 4700
 Connection ~ 6700 4700
-Wire Wire Line
-	7100 2600 7700 2600
-Wire Wire Line
-	7100 2500 7300 2500
-Wire Wire Line
-	7300 2500 7300 2350
-$Comp
-L GND #PWR09
-U 1 1 59807528
-P 7300 2900
-F 0 "#PWR09" H 7300 2650 50  0001 C CNN
-F 1 "GND" H 7300 2750 50  0000 C CNN
-F 2 "" H 7300 2900 50  0001 C CNN
-F 3 "" H 7300 2900 50  0001 C CNN
-	1    7300 2900
-	1    0    0    -1
-$EndComp
-Wire Wire Line
-	7100 2800 7300 2800
-Wire Wire Line
-	7300 2800 7300 2900
 $Comp
 L CONN_01X07 J1
@@
 Text Label 7700 2700 2    60   ~ 0
 V_BATT
+Text Label 5700 3300 2    60   ~ 0
+V_BATT
+Text Label 7700 2600 2    60   ~ 0
+V_BATT_EN
+Text Label 5700 3600 2    60   ~ 0
+V_BATT_EN
+Text Label 4900 3150 0    60   ~ 0
+~SS_EN
+Text Label 5700 3100 2    60   ~ 0
+~SS_EN
+Text Label 4900 3050 0    60   ~ 0
+SS_OUT
 Text Label 5700 3000 2    60   ~ 0
-V_BATT
-Wire Wire Line
-	4900 3150 5450 3150
-Wire Wire Line
-	5450 3150 5450 3600
-Wire Wire Line
-	5450 3600 5700 3600
+SS_OUT
+$Comp
+L DS18B20U U1
+U 1 1 59DE25EA
+P 3950 4050
+F 0 "U1" H 3800 4300 50  0000 C CNN
+F 1 "DS18B20U" H 4200 4300 50  0000 C CNN
+F 2 "Housings_SSOP:MSOP-8_3x3mm_Pitch0.65mm" H 3000 3800 50  0001 C CNN
+F 3 "" H 3800 4300 50  0001 C CNN
+	1    3950 4050
+	1    0    0    -1
+$EndComp
+Wire Wire Line
+	3950 3650 3950 3750
+Wire Wire Line
+	3950 4450 3950 4350
+Wire Wire Line
+	3950 4400 3650 4400
+Wire Wire Line
+	3650 4400 3650 3650
+Wire Wire Line
+	3650 3650 3950 3650
+Connection ~ 3950 4400
 $EndSCHEMATC

Commit message: update schematics
Connections:
- net VDD: no longer J1.3 (P3)
- new net VBUS: J1.3 (P3)
Changed lines of the file:
@@
 Connection ~ 5300 1600
-$Comp
-L VDD #PWR04
-U 1 1 5956777F
-P 4350 1750
-F 0 "#PWR04" H 4350 1600 50  0001 C CNN
-F 1 "VDD" H 4350 1900 50  0000 C CNN
-F 2 "" H 4350 1750 50  0001 C CNN
-F 3 "" H 4350 1750 50  0001 C CNN
-	1    4350 1750
-	1    0    0    -1
-$EndComp
 $Comp
 L GND #PWR05
@@
 	3650 3650 3950 3650
 Connection ~ 3950 4400
+$Comp
+L VBUS #PWR?
+U 1 1 59F88CC6
+P 4350 1750
+F 0 "#PWR?" H 4350 1600 50  0001 C CNN
+F 1 "VBUS" H 4350 1900 50  0000 C CNN
+F 2 "" H 4350 1750 50  0001 C CNN
+F 3 "" H 4350 1750 50  0001 C CNN
+	1    4350 1750
+	1    0    0    -1
+$EndComp
 $EndSCHEMATC

Commit message: update schematics
Parts:
- U1: symbol DS18B20U -> DS18B20U-RESCUE-soilsensor
Connections:
- net V_BATT_EN: now also U2.11 (P0.19); no longer U2.20 (P0.08)
Changed lines of the file:
@@
 Connection ~ 5300 1600
 $Comp
-L GND #PWR05
+L GND #PWR04
 U 1 1 595677AB
 P 3650 2050
-F 0 "#PWR05" H 3650 1800 50  0001 C CNN
+F 0 "#PWR04" H 3650 1800 50  0001 C CNN
 F 1 "GND" H 3650 1900 50  0000 C CNN
 F 2 "" H 3650 2050 50  0001 C CNN
@@
 $EndComp
 $Comp
-L GND #PWR06
+L GND #PWR05
 U 1 1 59567F04
 P 3950 4450
-F 0 "#PWR06" H 3950 4200 50  0001 C CNN
+F 0 "#PWR05" H 3950 4200 50  0001 C CNN
 F 1 "GND" H 3950 4300 50  0000 C CNN
 F 2 "" H 3950 4450 50  0001 C CNN
@@
 	4250 4050 5150 4050
 $Comp
-L VDD #PWR07
+L VDD #PWR06
 U 1 1 59568035
 P 4600 3550
-F 0 "#PWR07" H 4600 3400 50  0001 C CNN
+F 0 "#PWR06" H 4600 3400 50  0001 C CNN
 F 1 "VDD" H 4600 3700 50  0000 C CNN
 F 2 "" H 4600 3550 50  0001 C CNN
@@
 Text Label 7700 2600 2    60   ~ 0
 V_BATT_EN
-Text Label 5700 3600 2    60   ~ 0
+Text Label 7100 3400 0    60   ~ 0
 V_BATT_EN
 Text Label 4900 3150 0    60   ~ 0
@@
 SS_OUT
 $Comp
-L DS18B20U U1
+L DS18B20U-RESCUE-soilsensor U1
 U 1 1 59DE25EA
 P 3950 4050
@@
 Connection ~ 3950 4400
 $Comp
-L VBUS #PWR?
+L VBUS #PWR07
 U 1 1 59F88CC6
 P 4350 1750
-F 0 "#PWR?" H 4350 1600 50  0001 C CNN
+F 0 "#PWR07" H 4350 1600 50  0001 C CNN
 F 1 "VBUS" H 4350 1900 50  0000 C CNN
 F 2 "" H 4350 1750 50  0001 C CNN
