File: CapacitiveSoilSensor.sch (KiCad schematic (older format))
At the start: 13 parts, among them Q3 Q_PMOS_DGS, U5 TLC555

Commit message: fix cap. soil sensor
Parts:
- C10: footprint Capacitors_SMD:C_1206_HandSoldering -> Capacitors_SMD:C_0603
Changed lines of the file:
@@
 LIBS:rfcom
 LIBS:maxim
-LIBS:battery_management
+LIBS:sensors
+LIBS:Battery_Management
 LIBS:soilsensor-cache
 EELAYER 25 0
@@
 $EndComp
 $Comp
-L GND #PWR020
+L GND #PWR018
 U 1 1 59567668
 P 3400 3700
-F 0 "#PWR020" H 3400 3450 50  0001 C CNN
+F 0 "#PWR018" H 3400 3450 50  0001 C CNN
 F 1 "GND" H 3400 3550 50  0000 C CNN
 F 2 "" H 3400 3700 50  0001 C CNN
@@
 $EndComp
 $Comp
-L VDD #PWR021
+L VDD #PWR019
 U 1 1 5956766E
 P 3400 1600
-F 0 "#PWR021" H 3400 1450 50  0001 C CNN
+F 0 "#PWR019" H 3400 1450 50  0001 C CNN
 F 1 "VDD" H 3400 1750 50  0000 C CNN
 F 2 "" H 3400 1600 50  0001 C CNN
@@
 	2250 3250 2900 3250
 $Comp
-L GND #PWR022
+L GND #PWR020
 U 1 1 59567676
 P 2250 4250
-F 0 "#PWR022" H 2250 4000 50  0001 C CNN
+F 0 "#PWR020" H 2250 4000 50  0001 C CNN
 F 1 "GND" H 2250 4100 50  0000 C CNN
 F 2 "" H 2250 4250 50  0001 C CNN
@@
 F 0 "C10" H 5675 3100 50  0000 L CNN
 F 1 "1u" H 5675 2900 50  0000 L CNN
-F 2 "Capacitors_SMD:C_1206_HandSoldering" H 5688 2850 50  0001 C CNN
+F 2 "Capacitors_SMD:C_0603" H 5688 2850 50  0001 C CNN
 F 3 "" H 5650 3000 50  0001 C CNN
 	1    5650 3000
@@
 	4450 2800 4950 2800
 $Comp
-L GND #PWR023
+L GND #PWR021
 U 1 1 595676B6
 P 5350 3350
-F 0 "#PWR023" H 5350 3100 50  0001 C CNN
+F 0 "#PWR021" H 5350 3100 50  0001 C CNN
 F 1 "GND" H 5350 3200 50  0000 C CNN
 F 2 "" H 5350 3350 50  0001 C CNN
@@
 	3400 2300 3400 2850
 $Comp
-L VDD #PWR024
+L VDD #PWR022
 U 1 1 595A0C96
 P 4600 3150
-F 0 "#PWR024" H 4600 3000 50  0001 C CNN
+F 0 "#PWR022" H 4600 3000 50  0001 C CNN
 F 1 "VDD" H 4600 3300 50  0000 C CNN
 F 2 "" H 4600 3150 50  0001 C CNN
@@
 Connection ~ 3400 2450
 $Comp
-L GND #PWR025
+L GND #PWR023
 U 1 1 595676C9
 P 2450 2800
-F 0 "#PWR025" H 2450 2550 50  0001 C CNN
+F 0 "#PWR023" H 2450 2550 50  0001 C CNN
 F 1 "GND" H 2450 2650 50  0000 C CNN
 F 2 "" H 2450 2800 50  0001 C CNN
@@
 	4600 3250 4600 3150
 $Comp
-L GND #PWR026
+L GND #PWR024
 U 1 1 595676D9
 P 3950 4350
-F 0 "#PWR026" H 3950 4100 50  0001 C CNN
+F 0 "#PWR024" H 3950 4100 50  0001 C CNN
 F 1 "GND" H 3950 4200 50  0000 C CNN
 F 2 "" H 3950 4350 50  0001 C CNN
