File: CapacitiveSoilSensor.sch (KiCad schematic (older format))
At the start: 13 parts, among them Q3 Q_PMOS_DGS, U5 TLC555

Commit message: change mosfet layouts
Parts:
- removed Q3: Q_PMOS_DGS, TO_SOT_Packages_SMD:SOT-23, symbol Q_PMOS_DGS
- added Q?: Q_PMOS_GSD, symbol Q_PMOS_GSD
Changed lines of the file:
@@
 	4850 2850 4850 2800
 Connection ~ 4850 2800
-$Comp
-L Q_PMOS_DGS Q3
-U 1 1 59DCC707
-P 3300 2100
-F 0 "Q3" H 3500 2150 50  0000 L CNN
-F 1 "Q_PMOS_DGS" H 3500 2050 50  0000 L CNN
-F 2 "TO_SOT_Packages_SMD:SOT-23" H 3500 2200 50  0001 C CNN
-F 3 "" H 3300 2100 50  0001 C CNN
-	1    3300 2100
-	1    0    0    -1
-$EndComp
 Wire Wire Line
 	3400 1600 3400 1900
@@
 	2800 3450 2800 2450
 Connection ~ 2800 2450
+$Comp
+L Q_PMOS_GSD Q?
+U 1 1 59E47EF8
+P 3300 2100
+F 0 "Q?" H 3500 2150 50  0000 L CNN
+F 1 "Q_PMOS_GSD" H 3500 2050 50  0000 L CNN
+F 2 "" H 3500 2200 50  0001 C CNN
+F 3 "" H 3300 2100 50  0001 C CNN
+	1    3300 2100
+	1    0    0    -1
+$EndComp
 $EndSCHEMATC
