File: SoilMeasuringBoard.sch (KiCad schematic (older format))
At the start: 16 parts, among them J3 Conn_01x07, U1 RFD77101, U4 DS18B20U

Commit message: add flash memory
Parts:
- added C8: 0.1u, Capacitor_SMD:C_0603_1608Metric, symbol Device:C
- added R12, R13, R14: 100k, Resistor_SMD:R_0603_1608Metric, symbol Device:R
- added U5: SST26VF016B, Package_SO:SOIC-8_3.9x4.9mm_P1.27mm, symbol Memory_Flash:SST26VF016B
Connections:
- net labels added: SPI_MISO, SPI_MOSI, SPI_SCK, SPI_SS
- wire segments 67 -> 84
Changed lines of the file:
@@
 Text Label 7350 3950 2    50   ~ 0
 TEMP_EN
+$Comp
+L Memory_Flash:SST26VF016B U5
+U 1 1 5B619BAD
+P 10050 5700
+F 0 "U5" H 10350 5550 50  0000 L CNN
+F 1 "SST26VF016B" H 10350 5450 50  0000 L CNN
+F 2 "Package_SO:SOIC-8_3.9x4.9mm_P1.27mm" H 10150 5800 50  0001 C CNN
+F 3 "https://www.microchip.com/wwwproducts/en/SST26VF016B" H 10150 5800 50  0001 C CNN
+	1    10050 5700
+	1    0    0    -1
+$EndComp
+$Comp
+L Device:C C8
+U 1 1 5B619DAC
+P 10550 5350
+F 0 "C8" H 10665 5396 50  0000 L CNN
+F 1 "0.1u" H 10665 5305 50  0000 L CNN
+F 2 "Capacitor_SMD:C_0603_1608Metric" H 10588 5200 50  0001 C CNN
+F 3 "~" H 10550 5350 50  0001 C CNN
+	1    10550 5350
+	1    0    0    -1
+$EndComp
+Wire Wire Line
+	10250 5200 10250 5100
+Wire Wire Line
+	10250 5100 10550 5100
+Wire Wire Line
+	10550 5100 10550 5200
+$Comp
+L power:GND #PWR0105
+U 1 1 5B61B553
+P 10250 6200
+F 0 "#PWR0105" H 10250 5950 50  0001 C CNN
+F 1 "GND" H 10250 6050 50  0000 C CNN
+F 2 "" H 10250 6200 50  0001 C CNN
+F 3 "" H 10250 6200 50  0001 C CNN
+	1    10250 6200
+	1    0    0    -1
+$EndComp
+Wire Wire Line
+	10250 6100 10250 6200
+$Comp
+L power:GND #PWR0106
+U 1 1 5B61CD11
+P 10550 5500
+F 0 "#PWR0106" H 10550 5250 50  0001 C CNN
+F 1 "GND" H 10550 5350 50  0000 C CNN
+F 2 "" H 10550 5500 50  0001 C CNN
+F 3 "" H 10550 5500 50  0001 C CNN
+	1    10550 5500
+	1    0    0    -1
+$EndComp
+$Comp
+L Device:R R14
+U 1 1 5B61CF80
+P 9250 5150
+F 0 "R14" H 9320 5196 50  0000 L CNN
+F 1 "100k" H 9320 5105 50  0000 L CNN
+F 2 "Resistor_SMD:R_0603_1608Metric" V 9180 5150 50  0001 C CNN
+F 3 "~" H 9250 5150 50  0001 C CNN
+	1    9250 5150
+	1    0    0    -1
+$EndComp
+$Comp
+L Device:R R13
+U 1 1 5B61CFDC
+P 9000 5150
+F 0 "R13" H 9070 5196 50  0000 L CNN
+F 1 "100k" H 9070 5105 50  0000 L CNN
+F 2 "Resistor_SMD:R_0603_1608Metric" V 8930 5150 50  0001 C CNN
+F 3 "~" H 9000 5150 50  0001 C CNN
+	1    9000 5150
+	1    0    0    -1
+$EndComp
+$Comp
+L Device:R R12
+U 1 1 5B61D01A
+P 8750 5150
+F 0 "R12" H 8820 5196 50  0000 L CNN
+F 1 "100k" H 8820 5105 50  0000 L CNN
+F 2 "Resistor_SMD:R_0603_1608Metric" V 8680 5150 50  0001 C CNN
+F 3 "~" H 8750 5150 50  0001 C CNN
+	1    8750 5150
+	1    0    0    -1
+$EndComp
+$Comp
+L power:VDD #PWR0107
+U 1 1 5B61D0DE
+P 9000 4900
+F 0 "#PWR0107" H 9000 4750 50  0001 C CNN
+F 1 "VDD" H 9000 5050 50  0000 C CNN
+F 2 "" H 9000 4900 50  0001 C CNN
+F 3 "" H 9000 4900 50  0001 C CNN
+	1    9000 4900
+	1    0    0    -1
+$EndComp
+Wire Wire Line
+	8750 5000 8750 4950
+Wire Wire Line
+	8750 4950 9000 4950
+Wire Wire Line
+	9250 4950 9250 5000
+Wire Wire Line
+	9000 5000 9000 4950
+Connection ~ 9000 4950
+Wire Wire Line
+	9000 4950 9250 4950
+Wire Wire Line
+	9000 4900 9000 4950
+Wire Wire Line
+	9250 5300 9250 5400
+Wire Wire Line
+	9250 5400 9650 5400
+Wire Wire Line
+	9000 5300 9000 5800
+Wire Wire Line
+	9000 5800 9650 5800
+Wire Wire Line
+	8750 5300 8750 5900
+Wire Wire Line
+	8750 5900 9650 5900
+Text Label 9650 5400 1    50   ~ 0
+SPI_SS
+Text Label 9650 5500 2    50   ~ 0
+SPI_SCK
+Text Label 9650 5600 2    50   ~ 0
+SPI_MOSI
+Text Label 9650 5700 2    50   ~ 0
+SPI_MISO
+Text Label 8750 2850 0    50   ~ 0
+SPI_SCK
+Text Label 8750 3150 0    50   ~ 0
+SPI_MOSI
+Text Label 8750 2950 0    50   ~ 0
+SPI_MISO
+Text Label 8750 2650 0    50   ~ 0
+SPI_SS
+$Comp
+L power:VDD #PWR0108
+U 1 1 5B628D05
+P 10250 5000
+F 0 "#PWR0108" H 10250 4850 50  0001 C CNN
+F 1 "VDD" H 10250 5150 50  0000 C CNN
+F 2 "" H 10250 5000 50  0001 C CNN
+F 3 "" H 10250 5000 50  0001 C CNN
+	1    10250 5000
+	1    0    0    -1
+$EndComp
+Connection ~ 10250 5100
+Wire Wire Line
+	10250 5100 10250 5000
 $EndSCHEMATC
